File: kicad_Files/hammerhead.sch (KiCad schematic (older format))
At the start: 123 parts, among them J1 TYPE-C-31-M12_13, J5 Conn_01x06_Male, SW1 ESC, SW10 O, SW11 P, SW12 BKSP, SW13 TAB_125, SW14 A, SW15 S, SW16 D, SW17 F, SW18 G, SW19 H, SW2 Q, SW20 J, SW21 K, SW22 L, SW23 ENTER_175, SW24 LSHIFT_175, SW25 Z, SW26 X, SW27 C, SW28 V, SW29 B, SW3 W, SW30 N, SW31 M, SW32 /?, SW33 RSHIFT_125, SW34 FN_100, SW35 RSHIFT_225, SW36 SUPER_100, SW37 LALT_100, SW38 SPC_625, SW39 RALT_125, SW4 E, SW40 LCTRL_125, SW41 RCTRL_125, SW5 R, SW6 T, SW7 Y, SW8 U, SW9 I, U1 STM32F072-LQFP48, U2 USBLC6-2SC6, U3 MCP1700-3302E_SOT23

Commit message: Finished routing
Parts:
- removed CUSB1: 100n, Capacitor_SMD:C_0805_2012Metric_Pad1.15x1.40mm_HandSolder, symbol Device:C_Small
- added RF1: 10k, acheron_Components:R_SMD_1026, symbol Device:R_Small
- CSI1: value 100n -> 10u
- H5: symbol Mechanical:MountingHole -> Mechanical:MountingHole_Pad
- H7: symbol Mechanical:MountingHole_Pad -> Mechanical:MountingHole
- J5: symbol Connector:Conn_01x06_Male -> Connector:Conn_01x10_Male
- RCC1, RCC2: footprint acheron_Components:R_SMD_1026 -> Resistor_SMD:R_0402_1005Metric
- RD1: renamed from RSH2; footprint acheron_Components:R_SMD_1026 -> Resistor_SMD:R_0805_2012Metric
- RSH1: footprint acheron_Components:R_SMD_1026 -> Resistor_SMD:R_0805_2012Metric
- renumbered CSH2 to CD1, DSH1 to DD1
Connections:
- net Col12 is gone; now on net Col11: SW12.1 (Col)
- net 3.3V: now also J5.1 (Pin_1); no longer J5.6 (Pin_6)
- net 5V: now also RF1.2
- net BOOT0: now also J5.8 (Pin_8), RRST1.2, U1.44 (BOOT0); no longer J5.2 (Pin_2), RRST1.1
- net CASE: now also H5.1; no longer H7.1
- net Col1: now also U1.43 (2C1_SDA/PB7)
- net Col10: now also SW41.1 (Col), U1.46 (SPI2_NSS/I2S2_WS/I2C1_SDA/TIM17_CH1/PB9); no longer SW39.1 (Col)
- net Col11: now also U1.45 (I2C1_SCL/TIM16_CH1/PB8); no longer SW41.1 (Col)
- net Col2: now also U1.12 (PA2/ADC_IN2)
- net Col3: now also U1.11 (PA1/ADC_IN1)
- net Col4: now also U1.10 (PA0/ADC_IN0)
- net Col5: now also U1.6 (PF1/OSC_OUT)
- net Col6: now also U1.5 (PF0/OSC_IN)
- net Col7: now also U1.4 (PC15/OSC32_OUT)
- net Col8: now also U1.3 (PC14/OSC32_IN)
- net Col9: now also SW39.1 (Col), U1.2 (PC13)
- net GND: now also J5.3 (Pin_3), J5.9 (Pin_9), RRST1.1, RF1.1; no longer RRST1.2
- net NRST: now also J5.10 (Pin_10); no longer J5.1 (Pin_1)
- net Row1: now also U1.30 (TIM1_CH2/PA9); no longer D12.1 (K)
- net Row2: now also U1.42 (I2C1_SCL/PB6)
- net Row4: now also D12.1 (K), U1.13 (PA3/TIM15_CH2/ADC_IN3)
- net SWCLK: now also J5.4 (Pin_4); no longer J5.3 (Pin_3)
- net SWDIO: now also J5.2 (Pin_2); no longer J5.4 (Pin_4)
- net SWO: now reaches U1.31 (TIM1_CH3/PA10)
- net SWO: now also J5.6 (Pin_6)
- no-connect marks 2 -> 3
Other:
- moved on the sheet: CB1, CB2, CB3, CB4, CB5, CB6, CB7, CB8, D12, D39, D40, H6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

Commit message: Added extra pins breakouts
Parts:
- removed J5: Conn_01x06_Male, acheron_Connectors:HEADER_6PIN_HORIZONTAL, symbol Connector:Conn_01x10_Male
- added D43, D45: 1N4148, acheron_Components:D_SOD-123, symbol Device:D
- added J2: Conn_ARM_JTAG_SWD_10, acheron_Connectors:Conn_ARM_JTAG_SWD_10, symbol Connector:Conn_ARM_JTAG_SWD_10
- added J3: Conn_01x08, acheron_Connectors:PinHeader_1x8_P2.54mm_Vertical, symbol Connector_Generic:Conn_01x08
- added J4: Conn_01x08, acheron_Connectors:PinHeader_1x10_P2.54mm_Vertical, symbol Connector_Generic:Conn_01x10
- added SW42: LALT_125, acheron_MX_SolderMask:MX125, symbol acheronSymbols:MXSwitch
- added SW43: SPC_225, acheron_MX_SolderMask:MX225R, symbol acheronSymbols:MXSwitch
- added SW44: SPC_275, acheron_MX_SolderMask:MX275R, symbol acheronSymbols:MXSwitch
- added SW45: RALT_125, acheron_MX_SolderMask:MX125, symbol acheronSymbols:MXSwitch
- added SW46: SUPER_100, acheron_MX_SolderMask:MX100, symbol acheronSymbols:MXSwitch
Connections:
- net 3.3V: now also J2.1 (VTref)
- net Col1: now also U1.42 (I2C1_SCL/PB6); no longer U1.43 (2C1_SDA/PB7)
- net Col10: now also U1.4 (PC15/OSC32_OUT); no longer U1.46 (SPI2_NSS/I2S2_WS/I2C1_SDA/TIM17_CH1/PB9)
- net Col11: now also U1.3 (PC14/OSC32_IN); no longer U1.45 (I2C1_SCL/TIM16_CH1/PB8)
- net Col2: now also U1.15 (PA5/ADC_IN5/DAC_OUT2); no longer U1.12 (PA2/ADC_IN2)
- net Col3: now also U1.14 (PA4/TIM14_CH1/ADC_IN4), SW42.1 (Col); no longer U1.11 (PA1/ADC_IN1)
- net Col4: now also U1.13 (PA3/TIM15_CH2/ADC_IN3), SW44.1 (Col); no longer U1.10 (PA0/ADC_IN0)
- net Col5: now also U1.12 (PA2/ADC_IN2); no longer U1.6 (PF1/OSC_OUT)
- net Col6: now also U1.11 (PA1/ADC_IN1), SW43.1 (Col); no longer U1.5 (PF0/OSC_IN)
- net Col7: now also U1.10 (PA0/ADC_IN0); no longer U1.4 (PC15/OSC32_OUT)
- net Col8: now also U1.6 (PF1/OSC_OUT), SW45.1 (Col); no longer U1.3 (PC14/OSC32_IN)
- net Col9: now also U1.5 (PF0/OSC_IN), SW46.1 (Col); no longer U1.2 (PC13)
- net GND: now also J2.3 (GND), J2.5 (GND), J2.9 (GNDDetect)
- net NRST: now also J2.10 (~RESET~)
- net Row1: now also U1.43 (2C1_SDA/PB7); no longer U1.30 (TIM1_CH2/PA9)
- net Row2: now also U1.45 (I2C1_SCL/TIM16_CH1/PB8); no longer U1.42 (I2C1_SCL/PB6)
- net Row3: now also U1.2 (PC13)
- net Row4: now also U1.46 (SPI2_NSS/I2S2_WS/I2C1_SDA/TIM17_CH1/PB9), D43.1 (K), D45.1 (K); no longer U1.13 (PA3/TIM15_CH2/ADC_IN3)
- net SWCLK: now also J2.4 (SWDCLK/TCK)
- net SWDIO: now also J2.2 (SWDIO/TMS)
- net Extra18: now reaches U1.16 (PA6/ADC_IN6/TIM3_CH1/TIM16_CH1)
- net Extra18: now also J4.10 (Pin_10)
- net Extra17: now reaches U1.17 (PA7/TIM3_CH2/TIM14_CH1/ADC_IN7)
- net Extra17: now also J4.9 (Pin_9)
- net Extra16: now reaches U1.18 (PB0/TIM3_CH3/ADC_IN8)
- net Extra16: now also J4.8 (Pin_8)
- net Extra15: now reaches U1.19 (PB1/TIM3_CH4/TIM14_CH1/ADC_IN9)
- net Extra15: now also J4.7 (Pin_7)
- net Extra14: now reaches U1.20 (PB2)
- net Extra14: now also J4.6 (Pin_6)
- net Extra13: now reaches U1.21 (PB10/SPI2_SCK/I2C2_SCL/TIM2_CH3)
- net Extra13: now also J4.5 (Pin_5)
- net Extra12: now reaches U1.22 (PB11/TIM2_CH4/I2C2_SDA)
- net Extra12: now also J4.4 (Pin_4)
- net Extra11: now reaches U1.25 (PB12)
- net Extra11: now also J4.3 (Pin_3)
- net Extra10: now reaches U1.26 (SPI2_SCK/I2S2_CK/I2C2_SCL/PB13)
- net Extra10: now also J4.2 (Pin_2)
- net Extra9: now reaches U1.27 (PB14/SPI2_MISO/I2S2_MCK/I2C2_SDA/TIM15_CH1/PB15)
- net Extra9: now also J4.1 (Pin_1)
- net Extra8: now reaches U1.28 (SPI2_MOSI/I2S2_SD/PB15)
- net Extra8: now also J3.8 (Pin_8)
- net Extra7: now reaches U1.29 (TIM1_CH1/PA8)
- net Extra7: now also J3.7 (Pin_7)
- net Extra4: now reaches U1.38 (PA2)
- net Extra4: now also J3.4 (Pin_4)
- net Extra3: now reaches U1.39 (SPI1_SCK/I2S1_CK/TIM2_CH2/PB3)
- net Extra3: now also J3.3 (Pin_3)
- net Extra2: now reaches U1.40 (SPI1_MISO/I2S1_MCK/TIM3_CH1/PB4)
- net Extra2: now also J3.2 (Pin_2)
- net Extra1: now reaches U1.41 (SPI1_MOSI/I2S1_SD/TIM3_CH2/PB5)
- net Extra1: now also J3.1 (Pin_1)
- net at D37.2 (A), SW37.2 (Row): now also SW42.2 (Row)
- net at D38.2 (A), SW38.2 (Row): now also SW43.2 (Row)
- net at D39.2 (A), SW39.2 (Row): now also SW46.2 (Row)
- net SWO renamed Extra5
- net Extra5: now also J3.5 (Pin_5)
- new net: D43.2 (A), SW44.2 (Row)
- new net: D45.2 (A), SW45.2 (Row)
- new net Extra6: J3.6 (Pin_6), U1.30 (TIM1_CH2/PA9)
- no-connect marks 3 -> 4
Other:
- moved on the sheet: CD1, DD1, H5, H6, H7, RD1
