File: kicad_Files/hammerhead.kicad_pcb (KiCad board)
At the start: 2 copper layers, 228.6 x 77.5 mm, 123 parts, among them J1 TYPE-C-31-M12_13, J5 Conn_01x06_Male, SW1 ESC, SW10 O, SW11 P, SW12 BKSP, SW13 TAB_125, SW14 A, SW15 S, SW16 D, SW17 F, SW18 G, SW19 H, SW2 Q, SW20 J, SW21 K, SW22 L, SW23 ENTER_175, SW24 LSHIFT_175, SW25 Z, SW26 X, SW27 C, SW28 V, SW29 B, SW3 W, SW30 N, SW31 M, SW32 /?, SW33 RSHIFT_125, SW34 FN_100, SW35 RSHIFT_225, SW36 SUPER_100, SW37 LALT_100, SW38 SPC_625, SW39 RALT_125, SW4 E, SW40 LCTRL_125, SW41 RCTRL_125, SW5 R, SW6 T, SW7 Y, SW8 U, SW9 I, U1 STM32F072-LQFP48, U2 USBLC6-2SC6, U3 MCP1700-3302E_SOT23

Commit message: Finished routing
Parts:
- removed CUSB1: 100n, Capacitor_SMD:C_0805_2012Metric_Pad1.15x1.40mm_HandSolder
- added RF1: 10k, acheron_Components:R_SMD_1026, F.Cu at (155.4, 75.6)
- CSI1: value 100n -> 10u
- RCC1, RCC2: footprint acheron_Components:R_SMD_1026 -> Resistor_SMD:R_0402_1005Metric
- RD1: renamed from RSH2; footprint acheron_Components:R_SMD_1026 -> Resistor_SMD:R_0805_2012Metric
- RSH1: footprint acheron_Components:R_SMD_1026 -> Resistor_SMD:R_0805_2012Metric
- moved CB4 386.2 mm to (242.9, 93.7), turned to 180 degrees
- moved CB6 386.1 mm to (240.2, 103.6), turned to 90 degrees
- moved CB5 385.9 mm to (239.2, 103.6), turned to 90 degrees
- moved CB3 384.8 mm to (242.9, 92.7), turned to 180 degrees
- moved CB7 378.0 mm to (229.4, 93.7), turned to 90 degrees
- moved CB8 376.9 mm to (229.4, 91.6)
- moved CB1 376.3 mm to (227.5, 98.3), turned to 270 degrees
- moved CB2 376.3 mm to (228.5, 98.3), turned to 270 degrees
- moved CRST1 365.0 mm to (192.1, 75.8), turned to 270 degrees
- moved SWRST1 364.5 mm to (175.7, 75.6)
- moved RRST1 364.5 mm to (189.8, 75.7), turned to 270 degrees
- moved CRST2 359.4 mm to (184.9, 75.7), turned to 90 degrees
- moved DRST1 356.0 mm to (187.2, 75.7), turned to 270 degrees
- moved D1 347.0 mm to (262.6, 62.5), turned to 270 degrees
- moved D2 342.1 mm to (245.9, 62.5), turned to 270 degrees
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- renumbered CSH2 to CD1, DSH1 to DD1
Connections:
- D12 pad 1: Row1 -> Row4
- H5 pad 1: (no net) -> CASE
- H7 pad 1: CASE -> (no net)
- J5 pad 1: NRST -> 3.3V
- J5 pad 2: BOOT0 -> SWDIO
- J5 pad 3: SWCLK -> GND
- J5 pad 4: SWDIO -> SWCLK
- J5 pad 6: 3.3V -> SWO
- RRST1 pad 1: BOOT0 -> GND
- RRST1 pad 2: GND -> BOOT0
- SW12 pad 1: Col12 -> Col11
- SW39 pad 1: Col10 -> Col9
- SW41 pad 1: Col11 -> Col10
- U1 pad 10: Net-(U1-Pad10) -> Col4
- U1 pad 11: Net-(U1-Pad11) -> Col3
- U1 pad 12: Net-(U1-Pad12) -> Col2
- U1 pad 13: Net-(U1-Pad13) -> Row4
- U1 pad 2: Net-(U1-Pad2) -> Col9
- U1 pad 3: Net-(U1-Pad3) -> Col8
- U1 pad 30: Net-(U1-Pad30) -> Row1
- U1 pad 31: Net-(U1-Pad31) -> SWO
- U1 pad 4: Net-(U1-Pad4) -> Col7
- U1 pad 42: Net-(U1-Pad42) -> Row2
- U1 pad 43: Net-(U1-Pad43) -> Col1
- U1 pad 44: Net-(U1-Pad44) -> BOOT0
- U1 pad 45: Net-(U1-Pad45) -> Col11
- U1 pad 46: Net-(U1-Pad46) -> Col10
- U1 pad 5: Net-(U1-Pad5) -> Col6
- U1 pad 6: Net-(U1-Pad6) -> Col5
Routing:
- net Row4: track 0.00 -> 341.3 mm
- net Row1: track 0.00 -> 306.2 mm, vias 0 -> 2
- net Col11: track 0.00 -> 268.2 mm
- net Row2: track 0.00 -> 266.8 mm
- net Col10: track 0.00 -> 259.0 mm
- net Row3: track 0.00 -> 258.1 mm, vias 0 -> 2
- net Col9: track 0.00 -> 224.7 mm
- net 3.3V: track 0.00 -> 211.5 mm, vias 0 -> 7
- net D-: track 0.00 -> 194.0 mm
- net Col6: track 0.00 -> 187.2 mm
- net Col8: track 0.00 -> 174.3 mm
- net Col7: track 0.00 -> 153.8 mm
- net D+: track 0.00 -> 153.8 mm
- net NRST: track 0.00 -> 117.8 mm, vias 0 -> 3
- net Col5: track 0.00 -> 115.4 mm
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Other:
- net class Default: clearance 0.2 -> 0.127; trace_width 0.25 -> 0.254
- rule trace_clearance: 0.2 -> 0.127

Commit message: Added extra pins breakouts
Parts:
- removed J5: Conn_01x06_Male, acheron_Connectors:HEADER_6PIN_HORIZONTAL
- added D43: 1N4148, acheron_Components:D_SOD-123, F.Cu at (164.9, 119.7)
- added D45: 1N4148, acheron_Components:D_SOD-123, F.Cu at (103.0, 119.7)
- added J2: Conn_ARM_JTAG_SWD_10, acheron_Connectors:Conn_ARM_JTAG_SWD_10, F.Cu at (242.3, 124.5)
- added J3: Conn_01x08, acheron_Connectors:PinHeader_1x8_P2.54mm_Vertical, F.Cu at (263.0, 77.1)
- added J4: Conn_01x08, acheron_Connectors:PinHeader_1x10_P2.54mm_Vertical, F.Cu at (262.9, 113.8)
- added SW42: LALT_125, acheron_MX_SolderMask:MX125, F.Cu at (210.2, 124.5)
- added SW43: SPC_225, acheron_MX_SolderMask:MX225R, F.Cu at (124.5, 124.5)
- added SW44: SPC_275, acheron_MX_SolderMask:MX275R, F.Cu at (172.1, 124.5)
- added SW45: RALT_125, acheron_MX_SolderMask:MX125, F.Cu at (91.1, 124.5)
- added SW46: SUPER_100, acheron_MX_SolderMask:MX100, F.Cu at (69.7, 124.5)
- moved L2 85.1 mm to (239.9, 74.7)
- moved D13 15.5 mm to (244.7, 81.6)
- moved D35 11.9 mm to (253.0, 129.2), turned to 0 degrees
- moved L3 3.77 mm to (150.7, 93.5)
- moved D24 1.19 mm to (255.4, 109.0)
- moved CB1 0.77 mm to (227.4, 97.5)
- moved CB2 0.77 mm to (228.4, 97.5)
- moved CB7 0.77 mm to (229.3, 93.0), turned to 180 degrees
- moved CB8 0.18 mm to (229.3, 91.4)
Connections:
- U1 pad 10: Col4 -> Col7
- U1 pad 11: Col3 -> Col6
- U1 pad 12: Col2 -> Col5
- U1 pad 13: Row4 -> Col4
- U1 pad 14: Net-(U1-Pad14) -> Col3
- U1 pad 15: Net-(U1-Pad15) -> Col2
- U1 pad 16: Net-(U1-Pad16) -> Extra18
- U1 pad 17: Net-(U1-Pad17) -> Extra17
- U1 pad 18: Net-(U1-Pad18) -> Extra16
- U1 pad 19: Net-(U1-Pad19) -> Extra15
- U1 pad 2: Col9 -> Row3
- U1 pad 20: Net-(U1-Pad20) -> Extra14
- U1 pad 21: Net-(U1-Pad21) -> Extra13
- U1 pad 22: Net-(U1-Pad22) -> Extra12
- U1 pad 25: Net-(U1-Pad25) -> Extra11
- U1 pad 26: Net-(U1-Pad26) -> Extra10
- U1 pad 27: Net-(U1-Pad27) -> Extra9
- U1 pad 28: Net-(U1-Pad28) -> Extra8
- U1 pad 29: Net-(U1-Pad29) -> Extra7
- U1 pad 3: Col8 -> Col11
- U1 pad 30: Row1 -> Extra6
- U1 pad 31: SWO -> Extra5
- U1 pad 38: Net-(U1-Pad38) -> Extra4
- U1 pad 39: Net-(U1-Pad39) -> Extra3
- U1 pad 4: Col7 -> Col10
- U1 pad 40: Net-(U1-Pad40) -> Extra2
- U1 pad 41: Net-(U1-Pad41) -> Extra1
- U1 pad 42: Row2 -> Col1
- U1 pad 43: Col1 -> Row1
- U1 pad 45: Col11 -> Row2
- U1 pad 46: Col10 -> Row4
- U1 pad 5: Col6 -> Col9
- U1 pad 6: Col5 -> Col8
Routing:
- net Row4: track 341.3 -> 554.3 mm
- net Row3: track 258.1 -> 420.2 mm
- net D-: track 194.0 -> 141.4 mm, vias 0 -> 2
- net SWO: track 45.2 -> 0.00 mm, vias 1 -> 0
- net Extra18: track 0.00 -> 44.3 mm
- net NRST: track 117.8 -> 160.6 mm, vias 3 -> 2
- net Extra1: track 0.00 -> 42.5 mm
- net Extra17: track 0.00 -> 42.4 mm
- net Extra2: track 0.00 -> 40.1 mm
- net Col2: track 80.5 -> 120.2 mm
- net Extra16: track 0.00 -> 39.3 mm
- net Net-(U1-Pad14): track 39.2 -> 0.00 mm
- net Extra9: track 0.00 -> 38.6 mm
- net Net-(U1-Pad15): track 38.1 -> 0.00 mm
- net Extra15: track 0.00 -> 37.9 mm
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- added copper zone on B.Cu, net /SHIELD
Other:
- net class Default: clearance 0.127 -> 0.1524; trace_width 0.254 -> 0.1524; via_dia 0.8 -> 0.508; via_drill 0.4 -> 0.3048
- net class USB_Differential_Pair added: clearance 0.508, trace_width 0.1524, via_dia 0.508, via_drill 0.3048
- rule trace_clearance: 0.127 -> 0.1524
- rule trace_min: 0.2 -> 0.1524
- rule via_min_drill: 0.3 -> 0.3048
- rule via_min_size: 0.4 -> 0.508
- board text added: "(B1) 1.00U LALT"
- board text added: "(B1) 1.25U RALT"
- board text added: "(B1) 6.25U SPACE"
- board text added: "(B1) 6U SPACE STAB"
- board text added: "(B2) 1.25U LALT"
- board text added: "(B2) 1.25U RALT"
- board text added: "(B2) 1U GUI"
- board text added: "(B2) 2.25U SPACE"
- board text added: "(B2) 2.25U SPACE STAB"
- board text added: "(B2) 2.75U SPACE"
- board text added: "(B2) 2.75U SPACE STAB"
- board text added: "A10"
- board text added: "A2"
- board text added: "A6"
- board text added: "A7"
- board text added: "A8"
- board text added: "A9"
- board text added: "B0"
- board text added: "B1"
- board text added: "B10"
- board text added: "B11"
- board text added: "B12"
- board text added: "B13"
- board text added: "B14"
- board text added: "B15"
- board text added: "B3"
- board text added: "B4"
- board text added: "B5"

Commit message: Updated renders and README
Other:
- board text added: "(I) If you want to check or reroute a specific trace, it is recommended that you use the High Contrast mode. Turn it on at View > Contrast mode > Check "High Contrast Mode". The icon is also available at the left icon column."
- board text added: "(II) It is recommended that the user has some knowledge in Git usage, since it is the main VCS tool used for the Acheron Project."
- board text added: "(III) All footprints are available either through KiCad's native libraries or the Acheron Library (http://github.com/Gondolindrim/AcheronLibrary). To facilitate the portability of the Acheron projects, this library is generally added at the ${KIPRJMOD} folder as a Git submodule. Hence, right after cloning the PCB repository, run: $ git submodule init --update To update the submodules."
- board text added: "(IV) For detailed information, check the Acheron Docs page for the HammerheadPCB: http://gondolindrim.github.io/AcheronDocs/hammerhead/intro.html"
- board text added: "(i) The grid unit (1U) value used was 3/4" = 19.05mm"
- board text added: "(ii) The PCB was designed to fit the standards of the PCBWay manufacturer, at their cheapest settings."
- board text added: "(iii) All parts were quoted on the LCSC supplier (https://lcsc.com)."
- board text added: "(iv) You can always contact Gondolindrim through:"
- board text added: "(v) Most manufacturers list minimum character height as 0.8mm, and warn that any words using values below that will be undiscernable or unreadable. I have found that values down to 0.6mm (25 thou) can be used, although at that level a really close look is needed. Indeed, the minimum character height at which characters are easily readable is 0.8mm"
- board text added: "- Discord: Gondolindrim#9738"
- board text added: "- E-mail: alvaro.augusto.volpato@gmail.com"
- board text added: "- HammerheadPCB's GitHub page: http://github.com/Gondolindrim/Hammerhead"
- board text added: "- Reddit: /u/gondolindrim"
- board text added: "Also be sure to check with your parts supplier if they have all the necessary parts in the Bill of Materials and change parts and footprints accordingly to availability"
- board text added: "Be aware that capabilities may vary among manufacturers, so be sure to check with your manufacturer if they support the minimum values used."
- board text added: "GENERAL OBSERVATIONS"
- board text added: "HammerheadPCB V. pre-Alpha Designed by Gondolindrim "I dremel'd the PCB and it just doesn't work anymore""
- board text added: "MINIMUM CLEARANCE: 6 thou"
- board text added: "MINIMUM CLEARANCE: 8 thou"
- board text added: "MINIMUM VALUES"
- board text added: "RECOMMENDED VALUES"
- board text added: "SILKSCREEN CHARACTER HEIGHT: 25 thou (see General Observation (v))"
- board text added: "SILKSCREEN CHARACTER HEIGHT: 32 thou"
- board text added: "SILKSCREEN CHARACTER TRACE WIDTH: 6 thou"
- board text added: "SILKSCREEN CHARACTER TRACE WIDTH: 8 thou"
- board text added: "TRACE WIDTH: 10 thou"
- board text added: "TRACE WIDTH: 6 thou (approx. 0.15 mm)"
- board text added: "TRACE-TO-EDGE AND VIA-TO-EDGE DISTANCE: 8 thou"
- board text added: "These are general hints to use this PCB file. They are aimed specially at thoise new to KiCad or ECAD in general and to whoever wishes to use this project."
- board text added: "These values were the default values used when possible."
- board text added: "USAGE GUIDE (PLEASE READ)"
- board text added: "VIA DIAMETER: 20 thou (approx. 0.5mm)"
- board text added: "VIA DIAMETER: 32 thou (approx. 0.8mm)"
- board text added: "VIA HOLE SIZE: 12 thou (approx. 0.3mm)"
- board text added: "VIA HOLE SIZE: 16 thou (approx. 0.4mm)"
- board text added: "VIA-TO-VIA AND VIA-TO-TRACE CLEARANCE: 6 thou"
- board text added: "VIA-TO-VIA AND VIA-TO-TRACE CLEARANCE: 8 thou"
- board text removed: "(B1) 6.25U SPACE"
- board text removed: "(B1) 6U SPACE STAB"
- board text removed: "(B2) 2.25U SPACE"
- board text removed: "(B2) 2.25U SPACE STAB"
- board text removed: "(B2) 2.75U SPACE"
- board text removed: "(B2) 2.75U SPACE STAB"
